File: USB-6002-breakout-DIO.brd (EAGLE design)
At the start: 86.4 x 83.8 mm, 15 parts, among them P0.0 BNC-V, P0.1 BNC-V, P0.2 BNC-V, P0.3 BNC-V, P0.4 BNC-V, P0.5 BNC-V, P0.6 BNC-V, P0.7 BNC-V, P1.0 BNC-V, P1.1 BNC-V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

Commit message: routing cleanup
Routing:
- net P1.0: track 20.3 -> 34.6 mm, vias 1 -> 2
Changed lines of the file:
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@@
 <wire x1="1.27" y1="6.35" x2="1.27" y2="3.81" width="0.508" layer="20"/>
 <wire x1="1.27" y1="3.81" x2="6.35" y2="3.81" width="0.508" layer="20"/>
+<polygon width="0.127" layer="29">
+<vertex x="6.35" y="77.47"/>
+<vertex x="1.27" y="77.47"/>
+<vertex x="1.27" y="74.93"/>
+<vertex x="6.35" y="74.93"/>
+</polygon>
+<polygon width="0.127" layer="29">
+<vertex x="6.35" y="72.39"/>
+<vertex x="1.27" y="72.39"/>
+<vertex x="1.27" y="69.85"/>
+<vertex x="6.35" y="69.85"/>
+</polygon>
+<polygon width="0.127" layer="29">
+<vertex x="6.35" y="67.31"/>
+<vertex x="1.27" y="67.31"/>
+<vertex x="1.27" y="64.77"/>
+<vertex x="6.35" y="64.77"/>
+</polygon>
+<polygon width="0.127" layer="29">
+<vertex x="6.35" y="62.23"/>
+<vertex x="1.27" y="62.23"/>
+<vertex x="1.27" y="59.69"/>
+<vertex x="6.35" y="59.69"/>
+</polygon>
+<polygon width="0.127" layer="29">
+<vertex x="6.35" y="57.15"/>
+<vertex x="1.27" y="57.15"/>
+<vertex x="1.27" y="54.61"/>
+<vertex x="6.35" y="54.61"/>
+</polygon>
+<polygon width="0.127" layer="29">
+<vertex x="6.35" y="52.07"/>
+<vertex x="1.27" y="52.07"/>
+<vertex x="1.27" y="49.53"/>
+<vertex x="6.35" y="49.53"/>
+</polygon>
+<polygon width="0.127" layer="29">
+<vertex x="6.35" y="46.99"/>
+<vertex x="1.27" y="46.99"/>
+<vertex x="1.27" y="44.45"/>
+<vertex x="6.35" y="44.45"/>
+</polygon>
+<polygon width="0.127" layer="29">
+<vertex x="6.35" y="41.91"/>
+<vertex x="1.27" y="41.91"/>
+<vertex x="1.27" y="39.37"/>
+<vertex x="6.35" y="39.37"/>
+</polygon>
+<polygon width="0.127" layer="29">
+<vertex x="6.35" y="36.83"/>
+<vertex x="1.27" y="36.83"/>
+<vertex x="1.27" y="34.29"/>
+<vertex x="6.35" y="34.29"/>
+</polygon>
+<polygon width="0.127" layer="29">
+<vertex x="6.35" y="31.75"/>
+<vertex x="1.27" y="31.75"/>
+<vertex x="1.27" y="29.21"/>
+<vertex x="6.35" y="29.21"/>
+</polygon>
+<polygon width="0.127" layer="29">
+<vertex x="6.35" y="26.67"/>
+<vertex x="1.27" y="26.67"/>
+<vertex x="1.27" y="24.13"/>
+<vertex x="6.35" y="24.13"/>
+</polygon>
+<polygon width="0.127" layer="29">
+<vertex x="6.35" y="21.59"/>
+<vertex x="1.27" y="21.59"/>
+<vertex x="1.27" y="19.05"/>
+<vertex x="6.35" y="19.05"/>
+</polygon>
+<polygon width="0.127" layer="29">
+<vertex x="6.35" y="16.51"/>
+<vertex x="1.27" y="16.51"/>
+<vertex x="1.27" y="13.97"/>
+<vertex x="6.35" y="13.97"/>
+</polygon>
+<polygon width="0.127" layer="29">
+<vertex x="6.35" y="11.43"/>
+<vertex x="1.27" y="11.43"/>
+<vertex x="1.27" y="8.89"/>
+<vertex x="6.35" y="8.89"/>
+</polygon>
+<polygon width="0.127" layer="29">
+<vertex x="6.35" y="6.35"/>
+<vertex x="1.27" y="6.35"/>
+<vertex x="1.27" y="3.81"/>
+<vertex x="6.35" y="3.81"/>
+</polygon>
+<polygon width="0.127" layer="29">
+<vertex x="6.35" y="1.27"/>
+<vertex x="1.27" y="1.27"/>
+<vertex x="1.27" y="-1.27"/>
+<vertex x="6.35" y="-1.27"/>
+</polygon>
+<polygon width="0.127" layer="30">
+<vertex x="6.35" y="77.47"/>
+<vertex x="1.27" y="77.47"/>
+<vertex x="1.27" y="74.93"/>
+<vertex x="6.35" y="74.93"/>
+</polygon>
+<polygon width="0.127" layer="30">
+<vertex x="6.35" y="72.39"/>
+<vertex x="1.27" y="72.39"/>
+<vertex x="1.27" y="69.85"/>
+<vertex x="6.35" y="69.85"/>
+</polygon>
+<polygon width="0.127" layer="30">
+<vertex x="6.35" y="67.31"/>
+<vertex x="1.27" y="67.31"/>
+<vertex x="1.27" y="64.77"/>
+<vertex x="6.35" y="64.77"/>
+</polygon>
+<polygon width="0.127" layer="30">
+<vertex x="6.35" y="62.23"/>
+<vertex x="1.27" y="62.23"/>
+<vertex x="1.27" y="59.69"/>
+<vertex x="6.35" y="59.69"/>
+</polygon>
+<polygon width="0.127" layer="30">
+<vertex x="6.35" y="57.15"/>
+<vertex x="1.27" y="57.15"/>
+<vertex x="1.27" y="54.61"/>
+<vertex x="6.35" y="54.61"/>
+</polygon>
+<polygon width="0.127" layer="30">
+<vertex x="6.35" y="52.07"/>
+<vertex x="1.27" y="52.07"/>
+<vertex x="1.27" y="49.53"/>
+<vertex x="6.35" y="49.53"/>
+</polygon>
+<polygon width="0.127" layer="30">
+<vertex x="6.35" y="46.99"/>
+<vertex x="1.27" y="46.99"/>
+<vertex x="1.27" y="44.45"/>
+<vertex x="6.35" y="44.45"/>
+</polygon>
+<polygon width="0.127" layer="30">
+<vertex x="6.35" y="41.91"/>
+<vertex x="1.27" y="41.91"/>
+<vertex x="1.27" y="39.37"/>
+<vertex x="6.35" y="39.37"/>
+</polygon>
+<polygon width="0.127" layer="30">
+<vertex x="6.35" y="36.83"/>
+<vertex x="1.27" y="36.83"/>
+<vertex x="1.27" y="34.29"/>
+<vertex x="6.35" y="34.29"/>
+</polygon>
+<polygon width="0.127" layer="30">
+<vertex x="6.35" y="31.75"/>
+<vertex x="1.27" y="31.75"/>
+<vertex x="1.27" y="29.21"/>
+<vertex x="6.35" y="29.21"/>
+</polygon>
+<polygon width="0.127" layer="30">
+<vertex x="6.35" y="26.67"/>
+<vertex x="1.27" y="26.67"/>
+<vertex x="1.27" y="24.13"/>
+<vertex x="6.35" y="24.13"/>
+</polygon>
+<polygon width="0.127" layer="30">
+<vertex x="6.35" y="21.59"/>
+<vertex x="1.27" y="21.59"/>
+<vertex x="1.27" y="19.05"/>
+<vertex x="6.35" y="19.05"/>
+</polygon>
+<polygon width="0.127" layer="30">
+<vertex x="6.35" y="16.51"/>
+<vertex x="1.27" y="16.51"/>
+<vertex x="1.27" y="13.97"/>
+<vertex x="6.35" y="13.97"/>
+</polygon>
+<polygon width="0.127" layer="30">
+<vertex x="6.35" y="11.43"/>
+<vertex x="1.27" y="11.43"/>
+<vertex x="1.27" y="8.89"/>
+<vertex x="6.35" y="8.89"/>
+</polygon>
+<polygon width="0.127" layer="30">
+<vertex x="6.35" y="6.35"/>
+<vertex x="1.27" y="6.35"/>
+<vertex x="1.27" y="3.81"/>
+<vertex x="6.35" y="3.81"/>
+</polygon>
+<polygon width="0.127" layer="30">
+<vertex x="6.35" y="1.27"/>
+<vertex x="1.27" y="1.27"/>
+<vertex x="1.27" y="-1.27"/>
+<vertex x="6.35" y="-1.27"/>
+</polygon>
 </plain>
 <attributes>
@@
 <via x="11.43" y="35.56" extent="1-16" drill="0.35"/>
 <contactref element="P1.0" pad="1"/>
-<wire x1="11.43" y1="35.56" x2="24.13" y2="31.75" width="0" layer="19" extent="16-16"/>
+<wire x1="11.43" y1="35.56" x2="15.24" y2="31.75" width="0.508" layer="1"/>
+<wire x1="15.24" y1="31.75" x2="21.59" y2="31.75" width="0.508" layer="1"/>
+<via x="21.59" y="31.75" extent="1-16" drill="0.35"/>
+<wire x1="21.59" y1="31.75" x2="24.13" y2="31.75" width="0.508" layer="16"/>
 </signal>
 <signal name="P1.2">
